Commit message: Update roid1_urdf.urdf

File: URDF/roid1_urdf.urdf (robot description, URDF)
Before this commit: robot Roid1, 24 links, 19 joints
Links:
- removed link l_hipjointlower
- removed link l_hipjointupper
- removed link r_foot
- added link c_chest_b, mass 0.08659748664099903
- added link c_chest_c, mass 0.1751250442918052; collision mesh filename=package://roid1/URDF/roid1_description/meshes/c_chest_b.stl; visual mesh filename=package://roid1/URDF/roid1_description/meshes/c_chest_b.stl
- added link l_hipjoint_lower, mass 0.06689532645492419; collision mesh filename=package://roid1/URDF/roid1_description/meshes/l_hipjoint_lo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; visual mesh filename=package://roid1/URDF/roid1_description/meshes/l_hipjoint_lo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
- added link l_hipjoint_upper, mass 0.005702042499396512; collision mesh filename=package://roid1/URDF/roid1_description/meshes/l_hipjoint_up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; visual mesh filename=package://roid1/URDF/roid1_description/meshes/dec_l_hipjoin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
- added link r_foot_large, mass 0.03847104970565037; collision mesh filename=package://roid1/URDF/roid1_description/meshes/r_foot_large.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; visual mesh filename=package://roid1/URDF/roid1_description/meshes/r_foot_large.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
- link c_chest: mass None -> 0.033763915303500654; geometry visual mesh filename=package://roid1/URDF/roid1_description/meshes/c_chest.stl
- link c_head: mass None -> 0.012778861662402228
- link l_foot_large: mass None -> 0.03847104970565043
- link l_leg_lower: mass None -> 0.06094435150357522
- link l_leg_upper: mass None -> 0.09097466003274825
- link r_hipjoint_lower: mass None -> 0.0668953264549242
- link r_hipjoint_upper: mass None -> 0.005702042499396526
- link r_leg_lower: mass None -> 0.06094435150357523
- link r_leg_upper: mass None -> 0.09097466003274823
Joints:
- added joint c_chest_ab: type fixed, parent c_chest, child c_chest_b, origin xyz=0 0 0, limit lower=-3 upper=3 effort=0 velocity=0
- added joint c_chest_bc: type fixed, parent c_chest_b, child c_chest_c, origin xyz=0 0 0, limit lower=-3 upper=3 effort=0 velocity=0
- added joint l_hipjoint_roll: type revolute, parent l_hipjoint_upper, child l_hipjoint_lower, origin xyz=0 -0.004501 0, axis 1 0 0, limit lower=-3 upper=3 effort=0 velocity=0
- added joint l_hipjoint_yaw: type revolute, parent base_link, child l_hipjoint_upper, origin xyz=0.0 0.021530 -0.044936, axis 0 0 1, limit lower=-3 upper=3 effort=0 velocity=0
- added joint r_ankle_roll: type revolute, parent r_ankle, child r_foot_large, origin xyz=0.0 0.011404 -0.038550, axis 1 0 0, limit lower=-3 upper=3 effort=0 velocity=0
- joint r_hipjoint_yaw: parent c_waist -> base_link

Commit message: Update roid1_urdf.urdf

File: URDF/roid1_urdf.urdf (robot description, URDF)
Before this commit: robot Roid1, 26 links, 24 joints
Links:
- link l_leg_lower: geometry collision mesh filename=package://roid1/URDF/roid1_description/meshes/l_leg_lower_a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; collision mesh filename=package://roid1/URDF/roid1_description/meshes/l_leg_lower_b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
- link r_leg_lower: geometry collision mesh filename=package://roid1/URDF/roid1_description/meshes/r_leg_lower_a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; collision mesh filename=package://roid1/URDF/roid1_description/meshes/r_leg_lower_b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

Commit message: Upgrading to inatia include model.

File: URDF/roid1_urdf.urdf (robot description, URDF)
Before this commit: robot Roid1, 24 links, 23 joints
Links:
- removed link c_waist
- added link base_footprint
- added link c_chest_b, mass 0.08659748664099903
- added link c_chest_c, mass 0.1751250442918052; collision mesh filename=package://roid1/URDF/roid1_description/meshes/c_chest_b.stl; visual mesh filename=package://roid1/URDF/roid1_description/meshes/c_chest_b.stl
- link base_link: mass None -> 0.13408213174666955; geometry collision mesh filename=package://roid1/URDF/roid1_description/meshes/c_waist.stl; visual mesh filename=package://roid1/URDF/roid1_description/meshes/c_waist.stl
- link c_chest: mass None -> 0.033763915303500654; geometry visual mesh filename=package://roid1/URDF/roid1_description/meshes/c_chest.stl
- link c_head: mass None -> 0.012778861662402228; geometry collision mesh filename=package://roid1/URDF/roid1_description/meshes/c_head_a.stl; visual mesh filename=package://roid1/URDF/roid1_description/meshes/c_head_a.stl
- link l_ankle: mass None -> 0.06757551562559608; geometry collision mesh filename=package://roid1/URDF/roid1_description/meshes/l_ankle.stl; visual mesh filename=package://roid1/URDF/roid1_description/meshes/l_ankle.stl
- link l_elbow: mass None -> 0.044771268874731644; geometry collision mesh filename=package://roid1/URDF/roid1_description/meshes/l_elbow.stl; visual mesh filename=package://roid1/URDF/roid1_description/meshes/l_elbow.stl
- link l_foot_large: mass None -> 0.03847104970565043; geometry collision mesh filename=package://roid1/URDF/roid1_description/meshes/l_foot_large.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; visual mesh filename=package://roid1/URDF/roid1_description/meshes/l_foot_large.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
- link l_hipjoint_lower: mass None -> 0.06689532645492419; geometry collision mesh filename=package://roid1/URDF/roid1_description/meshes/l_hipjoint_lo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; visual mesh filename=package://roid1/URDF/roid1_description/meshes/l_hipjoint_lo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
- link l_hipjoint_upper: mass None -> 0.005702042499396512; geometry collision mesh filename=package://roid1/URDF/roid1_description/meshes/l_hipjoint_up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; visual mesh filename=package://roid1/URDF/roid1_description/meshes/dec_l_hipjoin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
- link l_leg_lower: mass None -> 0.06094435150357522; geometry collision mesh filename=package://roid1/URDF/roid1_description/meshes/l_leg_lower_a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; collision mesh filename=package://roid1/URDF/roid1_description/meshes/l_leg_lower_b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
- link l_leg_upper: mass None -> 0.09097466003274825; geometry collision mesh filename=package://roid1/URDF/roid1_description/meshes/l_leg_upper_a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; visual mesh filename=package://roid1/URDF/roid1_description/meshes/l_leg_upper_a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
- link l_lowerarm: mass None -> 0.02983803452815617; geometry collision mesh filename=package://roid1/URDF/roid1_description/meshes/l_arm_lower.s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; visual mesh filename=package://roid1/URDF/roid1_description/meshes/l_arm_lower.s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
- link l_shoulder: mass None -> 0.012120367829212707; geometry collision mesh filename=package://roid1/URDF/roid1_description/meshes/l_shoulder.stl; visual mesh filename=package://roid1/URDF/roid1_description/meshes/dec_shoulderp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
- link l_upperarm: mass None -> 0.09077338253436838; geometry collision mesh filename=package://roid1/URDF/roid1_description/meshes/l_arm_upper.s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; visual mesh filename=package://roid1/URDF/roid1_description/meshes/l_arm_upper.s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
- link r_ankle: mass None -> 0.06757551562559609; geometry collision mesh filename=package://roid1/URDF/roid1_description/meshes/r_ankle.stl; visual mesh filename=package://roid1/URDF/roid1_description/meshes/r_ankle.stl
- link r_elbow: mass None -> 0.044771268874731526; geometry collision mesh filename=package://roid1/URDF/roid1_description/meshes/r_elbow.stl; visual mesh filename=package://roid1/URDF/roid1_description/meshes/r_elbow.stl
- link r_foot_large: mass None -> 0.03847104970565037; geometry collision mesh filename=package://roid1/URDF/roid1_description/meshes/r_foot_large.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; visual mesh filename=package://roid1/URDF/roid1_description/meshes/r_foot_large.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
- link r_hipjoint_lower: mass None -> 0.0668953264549242; geometry collision mesh filename=package://roid1/URDF/roid1_description/meshes/r_hipjoint_lo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; visual mesh filename=package://roid1/URDF/roid1_description/meshes/r_hipjoint_lo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
- link r_hipjoint_upper: mass None -> 0.005702042499396526; geometry collision mesh filename=package://roid1/URDF/roid1_description/meshes/r_hipjoint_up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; visual mesh filename=package://roid1/URDF/roid1_description/meshes/dec_r_hipjoin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
- link r_leg_lower: mass None -> 0.06094435150357523; geometry collision mesh filename=package://roid1/URDF/roid1_description/meshes/r_leg_lower_a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; collision mesh filename=package://roid1/URDF/roid1_description/meshes/r_leg_lower_b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
- link r_leg_upper: mass None -> 0.09097466003274823; geometry collision mesh filename=package://roid1/URDF/roid1_description/meshes/r_leg_upper_a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; visual mesh filename=package://roid1/URDF/roid1_description/meshes/r_leg_upper_a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
- link r_lowerarm: mass None -> 0.029838034528201704; geometry collision mesh filename=package://roid1/URDF/roid1_description/meshes/r_arm_lower.s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; visual mesh filename=package://roid1/URDF/roid1_description/meshes/r_arm_lower.s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
- link r_shoulder: mass None -> 0.01212036782921271; geometry collision mesh filename=package://roid1/URDF/roid1_description/meshes/r_shoulder.stl; visual mesh filename=package://roid1/URDF/roid1_description/meshes/dec_shoulderp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
- link r_upperarm: mass None -> 0.09077338253436838; geometry collision mesh filename=package://roid1/URDF/roid1_description/meshes/r_arm_upper.s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; visual mesh filename=package://roid1/URDF/roid1_description/meshes/r_arm_upper.s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
Joints:
- removed joint c_waist_fixed
- added joint c_chest_ab: type fixed, parent c_chest, child c_chest_b, origin xyz=0 0 0, limit lower=-3 upper=3 effort=0 velocity=0
- added joint c_chest_bc: type fixed, parent c_chest_b, child c_chest_c, origin xyz=0 0 0, limit lower=-3 upper=3 effort=0 velocity=0
- joint c_chest_yaw: parent c_waist -> base_link
- joint l_hipjoint_yaw: parent c_waist -> base_link
- joint r_hipjoint_yaw: parent c_waist -> base_link

File: URDF/roid1_urdf_unity.urdf (robot description, URDF)
Before this commit: robot Roid1i, 24 links, 23 joints
Links:
- removed link l_foot_large
- removed link r_foot_large
- added link l_foot, mass 0.045; collision mesh filename=package://roid1_description/meshes/l_foot_large.stl; visual mesh filename=package://roid1_description/meshes/l_foot_large.stl
- added link r_foot, mass 0.045; collision mesh filename=package://roid1_description/meshes/r_foot_large.stl; visual mesh filename=package://roid1_description/meshes/r_foot_large.stl
- link c_chest: geometry collision mesh filename=package://roid1_description/meshes/c_chest.stl; visual mesh filename=package://roid1_description/meshes/c_chest_a.stl
- link l_leg_lower: geometry collision mesh filename=package://roid1_description/meshes/l_leg_lower.stl; collision mesh filename=package://roid1_description/meshes/l_leg_lower.stl
- link l_leg_upper: geometry collision mesh filename=package://roid1_description/meshes/l_leg_upper.stl; visual mesh filename=package://roid1_description/meshes/l_leg_upper_a.stl
- link r_leg_lower: geometry collision mesh filename=package://roid1_description/meshes/r_leg_lower.stl; visual mesh filename=package://roid1_description/meshes/r_leg_lower_a.stl
