Commit message: Update roid1_urdf_unity.urdf

File: URDF/roid1_urdf_unity.urdf (robot description, URDF)
Before this commit: robot Roid1, 26 links, 24 joints
Links:
- removed link base_footprint
- removed link c_chest_b
- removed link c_chest_c
- removed link l_foot_large
- removed link r_foot_large
- added link l_foot, mass 0.045; collision mesh filename=package://roid1_description/meshes/l_foot_large.stl; visual mesh filename=package://roid1_description/meshes/l_foot_large.stl
- added link r_foot, mass 0.045; collision mesh filename=package://roid1_description/meshes/r_foot_large.stl; visual mesh filename=package://roid1_description/meshes/r_foot_large.stl
- added link world
- link base_link: mass 0.13408213174666955 -> 0.1428
- link c_chest: mass 0.033763915303500654 -> 0.04215; geometry collision mesh filename=package://roid1_description/meshes/c_chest.stl; visual mesh filename=package://roid1_description/meshes/c_chest_a.stl
- link c_head: mass 0.012778861662402228 -> 0.013
- link l_ankle: mass 0.06757551562559608 -> 0.058
- link l_elbow: mass 0.044771268874731644 -> 0.044
- link l_hipjoint_lower: mass 0.06689532645492419 -> 0.058
- link l_hipjoint_upper: mass 0.005702042499396512 -> 0.0115
- link l_leg_lower: mass 0.06094435150357522 -> 0.061; geometry collision mesh filename=package://roid1_description/meshes/l_leg_lower.stl; collision mesh filename=package://roid1_description/meshes/l_leg_lower.stl
- link l_leg_upper: mass 0.09097466003274825 -> 0.091; geometry collision mesh filename=package://roid1_description/meshes/l_leg_upper.stl; visual mesh filename=package://roid1_description/meshes/l_leg_upper_a.stl
- link l_lowerarm: mass 0.02983803452815617 -> 0.030
- link l_shoulder: mass 0.012120367829212707 -> 0.014
- link l_upperarm: mass 0.09077338253436838 -> 0.098
- link r_ankle: mass 0.06757551562559609 -> 0.058
- link r_elbow: mass 0.044771268874731526 -> 0.044
- link r_hipjoint_lower: mass 0.0668953264549242 -> 0.058
- link r_hipjoint_upper: mass 0.005702042499396526 -> 0.0115
- link r_leg_lower: mass 0.06094435150357523 -> 0.061; geometry collision mesh filename=package://roid1_description/meshes/r_leg_lower.stl; visual mesh filename=package://roid1_description/meshes/r_leg_lower_a.stl
- link r_leg_upper: mass 0.09097466003274823 -> 0.091
- link r_lowerarm: mass 0.029838034528201704 -> 0.030
- link r_shoulder: mass 0.01212036782921271 -> 0.014
- link r_upperarm: mass 0.09077338253436838 -> 0.098
Joints:
- removed joint c_chest_ab
- removed joint c_chest_bc
- added joint fixed: type fixed, parent world, child base_link
- joint c_chest_yaw: limit lower=-3 upper=3 effort=0 velocity=0 -> lower=-3 upper=3 effort=1.373 velocity=7.48
- joint c_head_yaw: limit lower=-3 upper=3 effort=0 velocity=0 -> lower=-3 upper=3 effort=1.373 velocity=7.48
- joint l_ankle_pitch: limit lower=-3 upper=3 effort=0 velocity=0 -> lower=-3 upper=3 effort=1.373 velocity=7.48
- joint l_ankle_roll: limit lower=-3 upper=3 effort=0 velocity=0 -> lower=-3 upper=3 effort=1.373 velocity=7.48
- joint l_elbow_pitch: limit lower=-3 upper=3 effort=0 velocity=0 -> lower=-3 upper=3 effort=1.373 velocity=7.48
- joint l_elbow_yaw: limit lower=-3 upper=3 effort=0 velocity=0 -> lower=-3 upper=3 effort=1.373 velocity=7.48
- joint l_hipjoint_pitch: limit lower=-3 upper=3 effort=0 velocity=0 -> lower=-3 upper=3 effort=1.373 velocity=7.48
- joint l_hipjoint_roll: limit lower=-3 upper=3 effort=0 velocity=0 -> lower=-3 upper=3 effort=1.373 velocity=7.48
- joint l_hipjoint_yaw: limit lower=-3 upper=3 effort=0 velocity=0 -> lower=-3 upper=3 effort=1.373 velocity=7.48
- joint l_knee_pitch: limit lower=-3 upper=3 effort=0 velocity=0 -> lower=-3 upper=3 effort=1.373 velocity=7.48
- joint l_shoulder_pitch: limit lower=-3 upper=3 effort=0 velocity=0 -> lower=-3 upper=3 effort=1.373 velocity=7.48
- joint l_shoulder_roll: limit lower=-3 upper=3 effort=0 velocity=0 -> lower=-3 upper=3 effort=1.373 velocity=7.48
- joint r_ankle_pitch: limit lower=-3 upper=3 effort=0 velocity=0 -> lower=-3 upper=3 effort=1.373 velocity=7.48
- joint r_ankle_roll: limit lower=-3 upper=3 effort=0 velocity=0 -> lower=-3 upper=3 effort=1.373 velocity=7.48
- joint r_elbow_pitch: limit lower=-3 upper=3 effort=0 velocity=0 -> lower=-3 upper=3 effort=1.373 velocity=7.48
- joint r_elbow_yaw: limit lower=-3 upper=3 effort=0 velocity=0 -> lower=-3 upper=3 effort=1.373 velocity=7.48
- joint r_hipjoint_pitch: limit lower=-3 upper=3 effort=0 velocity=0 -> lower=-3 upper=3 effort=1.373 velocity=7.48
- joint r_hipjoint_roll: limit lower=-3 upper=3 effort=0 velocity=0 -> lower=-3 upper=3 effort=1.373 velocity=7.48
- joint r_hipjoint_yaw: limit lower=-3 upper=3 effort=0 velocity=0 -> lower=-3 upper=3 effort=1.373 velocity=7.48
- joint r_knee_pitch: limit lower=-3 upper=3 effort=0 velocity=0 -> lower=-3 upper=3 effort=1.373 velocity=7.48
- joint r_shoulder_pitch: limit lower=-3 upper=3 effort=0 velocity=0 -> lower=-3 upper=3 effort=1.373 velocity=7.48
- joint r_shoulder_roll: limit lower=-3 upper=3 effort=0 velocity=0 -> lower=-3 upper=3 effort=1.373 velocity=7.48

Commit message: Update roid1_urdf_unity.urdf
Fixed errors in the foot section.

File: URDF/roid1_urdf_unity.urdf (robot description, URDF)
Before this commit: robot Roid1i, 24 links, 23 joints
Joints:
- joint l_ankle_roll: child l_foot_large -> l_foot
- joint r_ankle_roll: child r_foot_large -> r_foot
